File: STM32F4_REV2.sch (KiCad schematic (older format))
At the start: 50 parts, among them J1 Screw_Terminal_01x02, J2 SWD, J3 Conn_01x04, J4 Conn_01x04, J5 USB_B_Micro, Q1 AO3401A, SW1 SW_SPDT, U1 MP2359DJ-LF-Z, U2 STM32F405RGT6, U3 USBLC6-2SC6, Y1 16MHz

Commit message: Updated the schematics and PCB
Parts:
- removed J1: Screw_Terminal_01x02, TerminalBlock_Phoenix:TerminalBlock_Phoenix_PT-1,5-2-3.5-H_1x02_P3.50mm_Horizontal, symbol Connector:Screw_Terminal_01x02
- removed J3, J4: Conn_01x04, Connector_Molex:Molex_PicoBlade_53048-0410_1x04_P1.25mm_Horizontal, symbol Connector_Generic:Conn_01x04
- removed Q1: AO3401A, Package_TO_SOT_SMD:SOT-23, symbol Transistor_FET:AO3401A
- added J1: Conn_01x22, Connector_PinHeader_2.54mm:PinHeader_1x22_P2.54mm_Horizontal, symbol Connector_Generic:Conn_01x22
- J5: symbol Connector:USB_B_Micro -> STM32F4_REV2-rescue:USB_B_Micro-Connector
- U1: symbol SchmillipKiCADLibrary:MP2359DJ-LF-Z -> STM32F4_REV2-rescue:MP2359DJ-LF-Z-SchmillipKiCADLibrary
Connections:
- net labels removed: +12V
- wire segments 139 -> 137
Changed lines of the file:
@@
 	1000 6750 1000 6650
 $Comp
-L SchmillipKiCADLibrary:MP2359DJ-LF-Z U1
+L STM32F4_REV2-rescue:MP2359DJ-LF-Z-SchmillipKiCADLibrary U1
 U 1 1 5F7EC586
 P 5825 1250
@@
 BUCK_FB
 $Comp
-L power:+12V #PWR02
-U 1 1 5F80C2E1
-P 750 900
-F 0 "#PWR02" H 750 750 50  0001 C CNN
-F 1 "+12V" H 750 1050 50  0000 C CNN
-F 2 "" H 750 900 50  0001 C CNN
-F 3 "" H 750 900 50  0001 C CNN
-	1    750  900
-	1    0    0    -1
-$EndComp
-$Comp
 L Device:Polyfuse_Small F1
 U 1 1 5F80C917
@@
 $EndComp
 $Comp
-L Transistor_FET:AO3401A Q1
-U 1 1 5F812F05
-P 1375 1275
-F 0 "Q1" V 1775 1275 50  0000 C CNN
-F 1 "AO3401A" V 1675 1275 50  0000 C CNN
-F 2 "Package_TO_SOT_SMD:SOT-23" H 1575 1200 50  0001 L CIN
-F 3 "http://www.aosmd.com/pdfs/datasheet/AO3401A.pdf" H 1375 1275 50  0001 L CNN
-F 4 "C15127" H 1375 1275 50  0001 C CNN "LCSC Part #"
-	1    1375 1275
-	0    -1   -1   0
-$EndComp
-$Comp
-L power:GND #PWR05
-U 1 1 5F816317
-P 1375 1475
-F 0 "#PWR05" H 1375 1225 50  0001 C CNN
-F 1 "GND" H 1375 1325 50  0000 C CNN
-F 2 "" H 1375 1475 50  0001 C CNN
-F 3 "" H 1375 1475 50  0001 C CNN
-	1    1375 1475
-	1    0    0    -1
-$EndComp
-$Comp
 L Device:Ferrite_Bead_Small FB1
 U 1 1 5F81A136
@@
 Text Notes 500  575  0    50   ~ 0
 Power Circuitry
-$Comp
-L Connector:Screw_Terminal_01x02 J1
-U 1 1 5F8DE78C
-P 6700 2850
-F 0 "J1" H 6800 2850 50  0000 L CNN
-F 1 "Screw_Terminal_01x02" H 6800 2750 50  0000 L CNN
-F 2 "TerminalBlock_Phoenix:TerminalBlock_Phoenix_PT-1,5-2-3.5-H_1x02_P3.50mm_Horizontal" H 6700 2850 50  0001 C CNN
-F 3 "~" H 6700 2850 50  0001 C CNN
-	1    6700 2850
-	1    0    0    -1
-$EndComp
-$Comp
-L power:GND #PWR020
-U 1 1 5F8DF6C8
-P 6500 2950
-F 0 "#PWR020" H 6500 2700 50  0001 C CNN
-F 1 "GND" H 6500 2800 50  0000 C CNN
-F 2 "" H 6500 2950 50  0001 C CNN
-F 3 "" H 6500 2950 50  0001 C CNN
-	1    6500 2950
-	1    0    0    -1
-$EndComp
-$Comp
-L power:+12V #PWR018
-U 1 1 5F8E1D17
-P 6500 2850
-F 0 "#PWR018" H 6500 2700 50  0001 C CNN
-F 1 "+12V" H 6500 3000 50  0000 C CNN
-F 2 "" H 6500 2850 50  0001 C CNN
-F 3 "" H 6500 2850 50  0001 C CNN
-	1    6500 2850
-	1    0    0    -1
-$EndComp
 $Comp
 L Connector_Generic:Conn_02x05_Odd_Even J2
@@
 	4825 7200 4825 6850
 $Comp
-L Connector_Generic:Conn_01x04 J3
-U 1 1 5F95A4AF
-P 6800 4150
-F 0 "J3" H 6900 4150 50  0000 L CNN
-F 1 "Conn_01x04" H 6900 4050 50  0000 L CNN
-F 2 "Connector_Molex:Molex_PicoBlade_53048-0410_1x04_P1.25mm_Horizontal" H 6800 4150 50  0001 C CNN
-F 3 "~" H 6800 4150 50  0001 C CNN
-	1    6800 4150
-	1    0    0    -1
-$EndComp
-$Comp
 L power:+3.3V #PWR027
 U 1 1 5F95B067
@@
 I2C1_SDA
 $Comp
-L Connector_Generic:Conn_01x04 J4
-U 1 1 5F95D55D
-P 9300 4150
-F 0 "J4" H 9400 4150 50  0000 L CNN
-F 1 "Conn_01x04" H 9400 4050 50  0000 L CNN
-F 2 "Connector_Molex:Molex_PicoBlade_53048-0410_1x04_P1.25mm_Horizontal" H 9300 4150 50  0001 C CNN
-F 3 "~" H 9300 4150 50  0001 C CNN
-	1    9300 4150
-	1    0    0    -1
-$EndComp
-$Comp
 L power:+3.3V #PWR028
 U 1 1 5F95DE4B
@@
 USART3_RX
 $Comp
-L Connector:USB_B_Micro J5
+L STM32F4_REV2-rescue:USB_B_Micro-Connector J5
 U 1 1 5F973FD8
 P 6775 5600
@@
 	2075 1175 1700 1175
 Connection ~ 1700 1175
-Wire Wire Line
-	1175 1175 750  1175
-Wire Wire Line
-	750  900  750  1175
+$Comp
+L Connector_Generic:Conn_01x22 J1
+U 1 1 60E3DF5B
+P 6650 2750
+F 0 "J1" H 6730 2742 50  0000 L CNN
+F 1 "Conn_01x22" H 6730 2651 50  0000 L CNN
+F 2 "Connector_PinHeader_2.54mm:PinHeader_1x22_P2.54mm_Horizontal" H 6650 2750 50  0001 C CNN
+F 3 "~" H 6650 2750 50  0001 C CNN
+	1    6650 2750
+	1    0    0    -1
+$EndComp
 $EndSCHEMATC

Commit message: Added some datasheets for thermocouple and updated schematics and PCB
Parts:
- removed J2: SWD, Connector_PinHeader_1.27mm:PinHeader_2x05_P1.27mm_Vertical_SMD, symbol Connector_Generic:Conn_02x05_Odd_Even
- removed SW1: SW_SPDT, Button_Switch_SMD:SW_SPDT_PCM12, symbol Switch:SW_SPDT
- added J2: Conn_ST_STDC14, Connector_PinHeader_1.27mm:PinHeader_2x07_P1.27mm_Vertical_SMD, symbol Connector:Conn_ST_STDC14
- added J3, J4, J6: Conn_01x04, Connector_PinHeader_2.54mm:PinHeader_1x04_P2.54mm_Vertical, symbol Connector_Generic:Conn_01x04
- added J7: Conn_01x06, Connector_PinHeader_2.54mm:PinHeader_1x06_P2.54mm_Vertical, symbol Connector_Generic:Conn_01x06
- added R12, R14, R16, R18, R20: 15k, Resistor_SMD:R_0603_1608Metric, symbol Device:R_Small
- added R13, R15, R17, R19, R23, R24: 10k, Resistor_SMD:R_0603_1608Metric, symbol Device:R_Small
- added R21: 1.5k, Resistor_SMD:R_0603_1608Metric, symbol Device:R_Small
- added R22: 1k, Resistor_SMD:R_0603_1608Metric, symbol Device:R_Small
- added SW1: SW_DIP_x01, Button_Switch_SMD:SW_DIP_SPSTx01_Slide_6.7x4.1mm_W6.73mm_P2.54mm_LowProfile_JPin, symbol Switch:SW_DIP_x01
- added U4: TXS0108EPWR, robot_regulator:SOP65P640X120-20N, symbol TXS0108EPWR:TXS0108EPWR
- added U5: TJA1051T, robot_regulator:SOT96-1, symbol TJA1051T:TJA1051T
- added U6, U7: TLP2361, TLP2361:SOIC-6-5_W4.55mm, symbol Interface_Optical_2:TLP2361
- J5: footprint SchmillipKiCADLibrary:USB_MICRO_B_101181930001LF -> USB_Micro-B_Molex_47346-0001:USB_Micro-B_Molex_47346-0001
- Y1: footprint Crystal:Crystal_SMD_3225-4Pin_3.2x2.5mm -> Oscillator:Oscillator_SMD_Abracon_ASE-4Pin_3.2x2.5mm
Connections:
- net +3V3: now also R7.1, J2.3 (VCC), J3.1 (Pin_1), J4.1 (Pin_1), J6.1 (Pin_1), J7.6 (Pin_6), R12.1, R22.1, R23.2, U4.2 (VCCA), U7.6 (VCC)
- net +5V: now also J1.1 (Pin_1), U4.19 (VCCB)
- net BOOT0: now also SW1.1
- net GND: now also J1.2 (Pin_2), J2.11 (GNDDetect), J2.5 (GND), J2.7 (GND), J3.4 (Pin_4), J4.4 (Pin_4), J6.4 (Pin_4), J7.5 (Pin_5), R14.2, R16.2, R18.2, R20.2, SW1.2, U4.11 (GND), U5.2 (GND), U5.8 (S), U7.4 (GND)
- net I2C1_SCL: now also J4.2 (Pin_2)
- net I2C1_SDA: now also J4.3 (Pin_3)
- net NRST: now also J2.12 (~RST)
- net SWCLK: now also J2.6 (JCLK/SWCLK)
- net SWDIO: now also J2.4 (JTMS/SWDIO)
- net SWO: now also J2.8 (JTDO/SWO)
- net USART3_RX: now also J6.3 (Pin_3)
- net USART3_TX: now also J6.2 (Pin_2)
- net A2: now reaches U2.10 (PC2)
- net A2: now also R17.2, R18.1
- net A3: now reaches U2.11 (PC3)
- net A3: now also R19.2, R20.1
- net THERMOCOUPLE_CS: now reaches U2.14 (PA0)
- net THERMOCOUPLE_CS: now also J7.1 (Pin_1)
- net DAC: now reaches U2.24 (PC4)
- net DAC: now also J1.7 (Pin_7)
- net ENABLEDISABLE: now reaches U2.26 (PB0)
- net ENABLEDISABLE: now also R12.2, U4.10 (OE)
- net CS: now reaches U2.33 (PB12)
- net CS: now also J1.13 (Pin_13)
- net SCK: now reaches U2.34 (PB13)
- net SCK: now also J1.14 (Pin_14), J7.4 (Pin_4)
- net MISO: now reaches U2.35 (PB14)
- net MISO: now also J1.16 (Pin_16), J7.3 (Pin_3)
- net MOSI: now reaches U2.36 (PB15)
- net MOSI: now also J1.15 (Pin_15)
- net INT: now reaches U2.37 (PC6)
- net INT: now also J1.12 (Pin_12)
- net COUT1: now reaches U2.38 (PC7)
- net COUT1: now also J1.17 (Pin_17)
- net COUT2: now reaches U2.39 (PC8)
- net COUT2: now also J1.18 (Pin_18)
- net CAN_RX: now reaches U2.61 (PB8)
- net CAN_RX: now also R23.1, U6.5 (Vo)
- net CAN_TX: now reaches U2.62 (PB9)
- net CAN_TX: now also U7.3 (Cathode)
- net A0: now reaches U2.8 (PC0)
- net A0: now also R13.2, R14.1
- net A1: now reaches U2.9 (PC1)
- net A1: now also R15.2, R16.1
- net A2_5: now reaches J1.10 (Pin_10)
- net A2_5: now also R17.1
- net A3_5: now reaches J1.11 (Pin_11)
- net A3_5: now also R19.1
- net ISO_5V: now reaches J1.19 (Pin_19)
- net ISO_5V: now also R21.1, R24.2, U6.6 (VCC)
- net ISO_GND: now reaches J1.20 (Pin_20)
- net ISO_GND: now also U6.4 (GND)
- net CANH: now reaches J1.21 (Pin_21)
- net CANH: now also J3.2 (Pin_2), U5.7 (CANH)
- net CANL: now reaches J1.22 (Pin_22)
- net CANL: now also J3.3 (Pin_3), U5.6 (CANL)
- net B5: now reaches J1.3 (Pin_3)
- net B5: now also U4.15 (B5)
- net B6: now reaches J1.4 (Pin_4)
- net B6: now also U4.14 (B6)
- net B7: now reaches J1.5 (Pin_5)
- net B7: now also U4.13 (B7)
- net B8: now reaches J1.6 (Pin_6)
- net B8: now also U4.12 (B8)
- net A0_5: now reaches J1.8 (Pin_8)
- net A0_5: now also R13.1
- net A1_5: now reaches J1.9 (Pin_9)
- net A1_5: now also R15.1
- new net: R21.2, U6.1 (Anode)
- new net: R22.2, U7.1 (Anode)
- new net B1: U4.20 (B1)
- new net B2: U4.18 (B2)
- new net B3: U4.17 (B3)
- new net B4: U4.16 (B4)
- new net ISO_CAN_RX: U5.4 (RXD), U6.3 (Cathode)
- new net ISO_CAN_TX: R24.1, U5.1 (TXD), U7.5 (Vo)
- no-connect marks 43 -> 28
Other:
- moved on the sheet: J1, J5, R7, U3
